File: board/pc_rev2/pcb/adc.kicad_sch (KiCad schematic)
At the start: 25 parts, among them J10 Conn_01x03, U4 LMV324B, U5 TC74HC4066AF, U6 LM331AU

Commit message: MSMP-IFを追加、スピーカ出力をOFFにする仕組みを追加（WIP）
Parts:
- removed J10: Conn_01x03, Connector_PinHeader_2.54mm:PinHeader_1x03_P2.54mm_Vertical, symbol Connector_Generic:Conn_01x03
Connections:
- net ain3: now also U5.11
Other:
- moved on the sheet: U5D
Changed lines of the file:
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@@
 	)
 	(junction
+		(at 58.42 63.5)
+		(diameter 0)
+		(color 0 0 0 0)
+	)
+	(junction
 		(at 149.86 96.52)
 		(diameter 0)
@@
 	)
 	(junction
-		(at 58.42 63.5)
-		(diameter 0)
-		(color 0 0 0 0)
-	)
-	(junction
 		(at 149.86 142.24)
 		(diameter 0)
@@
 	(wire
 		(pts
-			(xy 78.74 78.74) (xy 58.42 78.74)
-		)
-		(stroke
-			(width 0)
-			(type default)
-		)
-	)
-	(wire
-		(pts
 			(xy 170.18 93.98) (xy 170.18 97.79)
 		)
@@
 	(wire
 		(pts
-			(xy 38.1 96.52) (xy 71.12 96.52)
+			(xy 38.1 88.9) (xy 50.8 88.9)
 		)
 		(stroke
@@
 	(wire
 		(pts
-			(xy 78.74 88.9) (xy 78.74 78.74)
+			(xy 0.0762 7.6962) (xy 35.6362 7.6962)
 		)
 		(stroke
@@
 	(wire
 		(pts
-			(xy 172.72 39.37) (xy 172.72 44.45)
+			(xy 58.42 63.5) (xy 58.42 81.28)
 		)
 		(stroke
@@
 	(wire
 		(pts
-			(xy 109.22 142.24) (xy 114.3 142.24)
-		)
-		(stroke
-			(width 0)
-			(type default)
-		)
-	)
-	(wire
-		(pts
-			(xy 118.11 105.41) (xy 118.11 114.3)
+			(xy 172.72 39.37) (xy 172.72 44.45)
 		)
 		(stroke
@@
 	(wire
 		(pts
-			(xy 147.32 104.14) (xy 149.86 104.14)
+			(xy 35.6362 0.0762) (xy 35.6362 7.6962)
 		)
 		(stroke
@@
 	(wire
 		(pts
-			(xy 114.3 142.24) (xy 114.3 138.43)
+			(xy 109.22 142.24) (xy 114.3 142.24)
 		)
 		(stroke
@@
 	(wire
 		(pts
-			(xy 45.72 88.9) (xy 63.5 88.9)
+			(xy 118.11 105.41) (xy 118.11 114.3)
 		)
 		(stroke
@@
 	(wire
 		(pts
-			(xy 109.22 127) (xy 114.3 127)
+			(xy 147.32 104.14) (xy 149.86 104.14)
 		)
 		(stroke
@@
 	(wire
 		(pts
-			(xy 147.32 134.62) (xy 149.86 134.62)
+			(xy 114.3 142.24) (xy 114.3 138.43)
 		)
 		(stroke
@@
 	(wire
 		(pts
-			(xy 78.74 44.45) (xy 81.28 44.45)
+			(xy 109.22 127) (xy 114.3 127)
 		)
 		(stroke
@@
 	(wire
 		(pts
-			(xy 50.8 86.36) (xy 48.26 86.36)
+			(xy 147.32 134.62) (xy 149.86 134.62)
 		)
 		(stroke
@@
 	(wire
 		(pts
-			(xy 58.42 78.74) (xy 58.42 63.5)
+			(xy 78.74 44.45) (xy 81.28 44.45)
 		)
 		(stroke
@@
 	(wire
 		(pts
-			(xy 45.72 86.36) (xy 45.72 88.9)
-		)
-		(stroke
-			(width 0)
-			(type default)
-		)
-	)
-	(wire
-		(pts
 			(xy 38.1 63.5) (xy 43.18 63.5)
 		)
@@
 	(wire
 		(pts
-			(xy 43.18 88.9) (xy 38.1 88.9)
+			(xy 38.1 81.28) (xy 43.18 81.28)
 		)
 		(stroke
@@
 	(wire
 		(pts
-			(xy 43.18 86.36) (xy 43.18 88.9)
-		)
-		(stroke
-			(width 0)
-			(type default)
-		)
-	)
-	(wire
-		(pts
 			(xy 147.32 111.76) (xy 149.86 111.76)
 		)
@@
 	)
 	(label "vref"
-		(at 50.8 86.36 0)
-		(effects
-			(font
-				(size 1.27 1.27)
-			)
-			(justify left bottom)
-		)
-	)
-	(label "vref"
 		(at 152.4 88.9 0)
 		(effects
@@
 	(hierarchical_label "ain3"
 		(shape input)
-		(at 38.1 88.9 180)
+		(at 38.1 81.28 180)
 		(effects
 			(font
@@
 	(hierarchical_label "sel3"
 		(shape input)
-		(at 38.1 96.52 180)
+		(at 38.1 88.9 180)
 		(effects
 			(font
@@
 	(symbol
 		(lib_id "4xxx:4066")
-		(at 71.12 88.9 0)
+		(at 50.8 81.28 0)
 		(mirror x)
 		(unit 4)
@@
 		(dnp no)
 		(property "Reference" "U5"
-			(at 71.12 82.55 0)
+			(at 50.8 74.93 0)
 			(show_name no)
 			(do_not_autoplace no)
@@
 		)
 		(property "Value" "TC74HC4066AF"
-			(at 71.12 85.09 0)
+			(at 50.8 77.47 0)
 			(show_name no)
 			(do_not_autoplace no)
@@
 		)
 		(property "Footprint" "Package_SO:SO-14_5.3x10.2mm_P1.27mm"
-			(at 71.12 88.9 0)
+			(at 50.8 81.28 0)
 			(hide yes)
 			(show_name no)
@@
 		)
 		(property "Datasheet" "https://toshiba.semicon-storage.com/info/TC74HC4066AF_datasheet_en_20170130.pdf?did=16175&prodName=TC74HC4066AF"
-			(at 71.12 88.9 0)
+			(at 50.8 81.28 0)
 			(hide yes)
 			(show_name no)
@@
 		)
 		(property "Description" ""
-			(at 71.12 88.9 0)
+			(at 50.8 81.28 0)
 			(hide yes)
 			(show_name no)
@@
 					(unit 1)
 				)
-			)
-		)
-	)
-	(symbol
-		(lib_id "Connector_Generic:Conn_01x03")
-		(at 45.72 81.28 90)
-		(unit 1)
-		(body_style 1)
-		(exclude_from_sim no)
-		(in_bom yes)
-		(on_board yes)
-		(in_pos_files yes)
-		(dnp no)
-		(fields_autoplaced yes)
-		(property "Reference" "J10"
-			(at 45.72 74.93 90)
-			(show_name no)
-			(do_not_autoplace no)
-			(effects
-				(font
-					(size 1.27 1.27)
-				)
-			)
-		)
-		(property "Value" "Conn_01x03"
-			(at 45.72 77.47 90)
-			(show_name no)
-			(do_not_autoplace no)
-			(effects
-				(font
-					(size 1.27 1.27)
-				)
-			)
-		)
-		(property "Footprint" "Connector_PinHeader_2.54mm:PinHeader_1x03_P2.54mm_Vertical"
-			(at 45.72 81.28 0)
-			(hide yes)
-			(show_name no)
-			(do_not_autoplace no)
-			(effects
-				(font
-					(size 1.27 1.27)
-				)
-			)
-		)
-		(property "Datasheet" ""
-			(at 45.72 81.28 0)
-			(hide yes)
-			(show_name no)
-			(do_not_autoplace no)
-			(effects
-				(font
-					(size 1.27 1.27)
-				)
-			)
-		)
-		(property "Description" "Generic connector, single row, 01x03, script generated (kicad-library-utils/schlib/autogen/connector/)"
-			(at 45.72 81.28 0)
-			(hide yes)
-			(show_name no)
-			(do_not_autoplace no)
-			(effects
-				(font
-					(size 1.27 1.27)
-				)
-			)
-		)
-		(pin "1"
-		)
-		(pin "2"
-		)
-		(pin "3"
-		)
-		(instances
-			(project "pc_rev2"
-				(path "/504622d4-653f-4b3b-8099-0af1a54c930d/7b66336c-3b34-40c8-983a-3c783378ed55"
-					(reference "J10")
-					(unit 1)
-				)

Commit message: ADCの8ch化＆スピーカーミュートの仕組み変更
Parts:
- removed unit 4 of U5
- removed unit 2 of U5
- removed unit 3 of U5
- added U8: 74HC4051, symbol 74xx:74HC4051
Connections:
- net +3.3V: now also U8.16 (VCC)
- net GND: now also U8.6 (~{E}), U8.7 (VEE), U8.8 (GND)
- net ain1: now also U8.14 (A1)
- net ain2: now also U8.15 (A2)
- net ain3: now also U8.12 (A3)
- net sel1: now also U8.10 (S1)
- net sel2: now also U8.9 (S2)
- net at U4.5 (+): now also U8.3 (A)
- net vref: no longer names the net of R17.2, R18.2, U4.10 (+), U6.1 (-)
- new net ain0: U8.13 (A0)
- new net ain4: U8.1 (A4)
- new net ain5: U8.5 (A5)
- new net ain6: U8.2 (A6)
- new net ain7: U8.4 (A7)
- new net sel0: U8.11 (S0)
Other:
- moved on the sheet: C11, U4A, U4B, U5A

Commit message: 諸々改良＆基板デザイン（WIP）
Parts:
- removed R16: 10k, Resistor_SMD:R_0603_1608Metric_Pad0.98x0.95mm_HandSolder, symbol Device:R
- added C15, C16: 100nF, Capacitor_SMD:C_0603_1608Metric_Pad1.08x0.95mm_HandSolder, symbol Device:C
- added U10: MCP1501-30xCH, Package_TO_SOT_SMD:SOT-23-6, symbol Reference_Voltage:MCP1501-30xCH
- added unit 4 of U5
- added unit 3 of U5
- U4: Manufacturer (none) -> 3PEAK; Manufacturer PN (none) -> LMV324B-TR
- U6: value LM331AU -> TPCMP231; symbol uchan:NJU7109 -> Comparator:MCP6561-OT; Manufacturer (none) -> 3PEAK; Manufacturer PN (none) -> TPCMP231-S5TR
- U8: footprint (none) -> Package_SO:SOIC-16W_5.3x10.2mm_P1.27mm; Manufacturer (none) -> Toshiba; Manufacturer PN (none) -> TC74HC4051AF(EL,F)
Connections:
- net ain6 is gone; now on net dac_out: U8.2 (A6)
- net +3.3V: now also C10.1, U6.5 (V+), C16.1
- net +5V: now also C15.1, U10.4 (~{SHDN}), U10.6 (VDD); no longer C10.1, U6.5 (V+)
- net GND: now also U4.5 (+), C15.2, C16.2, U10.2 (GND), U10.3 (GND), U10.5 (GND), U5.10, U5.11, U5.12, U5.6, U5.8, U5.9; no longer U4.12 (+)
- net ain_buf: now also U4.8, U4.9 (-), U5.3; no longer U4.6 (-), U4.7, U5.1
- net cmp: now also U6.1; no longer U6.4
- net dac_out: now also U4.13 (-), U4.14; no longer U4.8, U4.9 (-)
- net sh_buf: now also U4.2 (-); no longer U4.3 (+)
- net sh_on: now also U5.5; no longer U5.13
- net dac_raw: now reaches R17.2, R18.2
- net dac_raw: now also U4.12 (+), U6.4 (-); no longer U4.10 (+), U6.1 (-)
- net at U8.3 (A): now also U4.10 (+); no longer U4.5 (+)
- net ain7: no longer names the net of U8.4 (A7)
- net ain7: now also U10.1 (OUT)
- new net: C11.1, U4.3 (+), U5.4
- new net: U4.6 (-), U4.7
Other:
- note added: "3.0V"
- note added: "プッシュプル出力 レールツーレール出力"
- note removed: "オープンコレクタ出力"
