File: board/pc_rev2/pcb/msmp.kicad_sch (KiCad schematic)
At the start: 9 parts, among them J15 INPUT, J16 OUTPUT, U9 TLP2361

Commit message: 諸々改良＆基板デザイン（WIP）
Parts:
- added J21: Conn_Grove_Host, uchan:Grove_1x04_P2mm_THT_Horizontal, symbol uchan:Conn_Grove_Host
- R33: value 220 -> 390; footprint Resistor_THT:R_Axial_DIN0207_L6.3mm_D2.5mm_P7.62mm_Horizontal -> uchan:R_Axial_CF25_CFS50_L6.3mm_D2.3mm_P7.62mm_Horizontal; Manufacturer PN (none) -> CF25J390RB
- R34: footprint Resistor_THT:R_Axial_DIN0207_L6.3mm_D2.5mm_P7.62mm_Horizontal -> uchan:R_Axial_CF25_CFS50_L6.3mm_D2.3mm_P7.62mm_Horizontal; Manufacturer (none) -> FAITHFUL LINK INDUSTRIAL; Manufacturer PN (none) -> CFS50J33RB
- R35: footprint Resistor_THT:R_Axial_DIN0207_L6.3mm_D2.5mm_P7.62mm_Horizontal -> uchan:R_Axial_CF25_CFS50_L6.3mm_D2.3mm_P7.62mm_Horizontal; Manufacturer (none) -> FAITHFUL LINK INDUSTRIAL; Manufacturer PN (none) -> CF25J10RB
- U9: footprint Package_SO:SO-5_4.4x3.6mm_P1.27mm -> Package_SO:SO-5-6_4.55x3.7mm_P1.27mm
Connections:
- net GND: now also J21.4 (GND)
- net msmp_rx: now also J21.1 (RX)
- net msmp_tx: now also J21.2 (TX)
- new net +5V: J21.3 (VCC)
