File: board/pc_rev2/pcb/mcu.kicad_sch (KiCad schematic)
At the start: 2 parts, among them U1 Tang_nano_9K, U7 Tang_nano_20K

Commit message: ADCの8ch化＆スピーカーミュートの仕組み変更
Connections:
- net adc_sel3 is gone; now on net adc_sel2: U1.22 (PIN57_IOR13A), U7.3 (PIN75_IOT34A)
- net adc_sel1: now also U1.21 (PIN56_IOR14A), U7.2 (PIN74_IOT34B); no longer U1.20 (PIN55_IOR14B), U7.1 (PIN73_IOT40A)
- net adc_sel2: no longer U1.21 (PIN56_IOR14A), U7.2 (PIN74_IOT34B)
- net spk_on: now reaches U7.32 (PIN51_IOR45A)
- net spk_on: now also U1.17 (PIN51_IOR17B)
- new net adc_sel0: U1.20 (PIN55_IOR14B), U7.1 (PIN73_IOT40A)
- no-connect marks 10 -> 8
Changed lines of the file:
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@@
-	)
-	(no_connect
-		(at 134.62 121.92)
 	)
 	(no_connect
@@
 	(no_connect
 		(at 134.62 27.94)
-	)
-	(no_connect
-		(at 63.5 66.04)
 	)
 	(no_connect
@@
 		)
 	)
-	(hierarchical_label "adc_sel3"
-		(shape output)
-		(at 63.5 106.68 180)
-		(effects
-			(font
-				(size 1.27 1.27)
-			)
-			(justify right)
-		)
-	)
 	(hierarchical_label "adc_sel2"
 		(shape output)
+		(at 63.5 78.74 180)
+		(effects
+			(font
+				(size 1.27 1.27)
+			)
+			(justify right)
+		)
+	)
+	(hierarchical_label "adc_vref_d2"
+		(shape output)
+		(at 63.5 40.64 180)
+		(effects
+			(font
+				(size 1.27 1.27)
+			)
+			(justify right)
+		)
+	)
+	(hierarchical_label "gpio4"
+		(shape output)
+		(at 63.5 142.24 180)
+		(effects
+			(font
+				(size 1.27 1.27)
+			)
+			(justify right)
+		)
+	)
+	(hierarchical_label "adc_sel0"
+		(shape output)
+		(at 63.5 73.66 180)
+		(effects
+			(font
+				(size 1.27 1.27)
+			)
+			(justify right)
+		)
+	)
+	(hierarchical_label "tf_mosi"
+		(shape output)
+		(at 63.5 27.94 180)
+		(effects
+			(font
+				(size 1.27 1.27)
+			)
+			(justify right)
+		)
+	)
+	(hierarchical_label "adc_vref_d2"
+		(shape output)
+		(at 63.5 121.92 180)
+		(effects
+			(font
+				(size 1.27 1.27)
+			)
+			(justify right)
+		)
+	)
+	(hierarchical_label "spk_on"
+		(shape output)
+		(at 63.5 66.04 180)
+		(effects
+			(font
+				(size 1.27 1.27)
+			)
+			(justify right)
+		)
+	)
+	(hierarchical_label "adc_vref_d5"
+		(shape output)
+		(at 63.5 129.54 180)
+		(effects
+			(font
+				(size 1.27 1.27)
+			)
+			(justify right)
+		)
+	)
+	(hierarchical_label "gpio2"
+		(shape output)
+		(at 63.5 137.16 180)
+		(effects
+			(font
+				(size 1.27 1.27)
+			)
+			(justify right)
+		)
+	)
+	(hierarchical_label "gpio1"
+		(shape output)
+		(at 63.5 116.84 180)
+		(effects
+			(font
+				(size 1.27 1.27)
+			)
+			(justify right)
+		)
+	)
+	(hierarchical_label "adc_sel1"
+		(shape output)
 		(at 63.5 76.2 180)
-		(effects
-			(font
-				(size 1.27 1.27)
-			)
-			(justify right)
-		)
-	)
-	(hierarchical_label "adc_vref_d2"
-		(shape output)
-		(at 63.5 40.64 180)
-		(effects
-			(font
-				(size 1.27 1.27)
-			)
-			(justify right)
-		)
-	)
-	(hierarchical_label "gpio4"
-		(shape output)
-		(at 63.5 142.24 180)
-		(effects
-			(font
-				(size 1.27 1.27)
-			)
-			(justify right)
-		)
-	)
-	(hierarchical_label "adc_sel3"
-		(shape output)
-		(at 63.5 78.74 180)
-		(effects
-			(font
-				(size 1.27 1.27)
-			)
-			(justify right)
-		)
-	)
-	(hierarchical_label "tf_mosi"
-		(shape output)
-		(at 63.5 27.94 180)
-		(effects
-			(font
-				(size 1.27 1.27)
-			)
-			(justify right)
-		)
-	)
-	(hierarchical_label "adc_vref_d2"
-		(shape output)
-		(at 63.5 121.92 180)
-		(effects
-			(font
-				(size 1.27 1.27)
-			)
-			(justify right)
-		)
-	)
-	(hierarchical_label "adc_vref_d5"
-		(shape output)
-		(at 63.5 129.54 180)
-		(effects
-			(font
-				(size 1.27 1.27)
-			)
-			(justify right)
-		)
-	)
-	(hierarchical_label "gpio2"
-		(shape output)
-		(at 63.5 137.16 180)
-		(effects
-			(font
-				(size 1.27 1.27)
-			)
-			(justify right)
-		)
-	)
-	(hierarchical_label "gpio1"
-		(shape output)
-		(at 63.5 116.84 180)
-		(effects
-			(font
-				(size 1.27 1.27)
-			)
-			(justify right)
-		)
-	)
-	(hierarchical_label "adc_sel1"
-		(shape output)
-		(at 63.5 73.66 180)
 		(effects
 			(font
@@
 		)
 	)
+	(hierarchical_label "adc_sel2"
+		(shape output)
+		(at 63.5 106.68 180)
+		(effects
+			(font
+				(size 1.27 1.27)
+			)
+			(justify right)
+		)
+	)
 	(hierarchical_label "tf_miso"
 		(shape output)
 		(at 63.5 33.02 180)
-		(effects
-			(font
-				(size 1.27 1.27)
-			)
-			(justify right)
-		)
-	)
-	(hierarchical_label "adc_sel2"
-		(shape output)
-		(at 63.5 104.14 180)
 		(effects
 			(font
@@
 		)
 	)
+	(hierarchical_label "adc_sel1"
+		(shape output)
+		(at 63.5 104.14 180)
+		(effects
+			(font
+				(size 1.27 1.27)
+			)
+			(justify right)
+		)
+	)
 	(hierarchical_label "adc_vref_d4"
 		(shape output)
@@
 			)
 			(justify left)
+		)
+	)
+	(hierarchical_label "adc_sel0"
+		(shape output)
+		(at 63.5 101.6 180)
+		(effects
+			(font
+				(size 1.27 1.27)
+			)
+			(justify right)
 		)
 	)
@@
 		)
 	)
+	(hierarchical_label "spk_on"
+		(shape output)
+		(at 134.62 121.92 0)
+		(effects
+			(font
+				(size 1.27 1.27)
+			)
+			(justify left)
+		)
+	)
 	(hierarchical_label "gpio5"
 		(shape output)
@@
 		)
 	)
-	(hierarchical_label "adc_sel1"
-		(shape output)
-		(at 63.5 101.6 180)
-		(effects
-			(font
-				(size 1.27 1.27)
-			)
-			(justify right)
-		)
-	)

Commit message: 諸々改良＆基板デザイン（WIP）
Parts:
- U7: now not fitted
Connections:
- net edid_clk is gone; now on net scl: U7.22 (PIN53_IOR38B)
- net adc_sel0: now also U1.15 (PIN41_IOB41A); no longer U1.20 (PIN55_IOR14B)
- net adc_sel1: now also U1.16 (PIN42_IOB41B); no longer U1.21 (PIN56_IOR14A)
- net adc_sel2: now also U1.17 (PIN51_IOR17B); no longer U1.22 (PIN57_IOR13A)
- net spk_on: now also U1.18 (PIN53_IOR15B); no longer U1.17 (PIN51_IOR17B)
- net uart2_rx: now also U1.20 (PIN55_IOR14B); no longer U1.16 (PIN42_IOB41B)
- net uart2_tx: now also U1.19 (PIN54_IOR15A); no longer U1.15 (PIN41_IOB41A)
- net uart_rx: now also U1.22 (PIN57_IOR13A); no longer U1.19 (PIN54_IOR15A)
- net uart_tx: now also U1.21 (PIN56_IOR14A); no longer U1.18 (PIN53_IOR15B)
- net scl: now reaches U1.47 (PIN86_IOT8A)
- net dbgio3 renamed sda
- no-connect marks 8 -> 7
Changed lines of the file:
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@@
-	)
-	(no_connect
-		(at 134.62 27.94)
 	)
 	(no_connect
@@
 	(hierarchical_label "adc_sel2"
 		(shape output)
-		(at 63.5 78.74 180)
+		(at 63.5 66.04 180)
 		(effects
 			(font
@@
 	(hierarchical_label "adc_sel0"
 		(shape output)
-		(at 63.5 73.66 180)
+		(at 63.5 60.96 180)
 		(effects
 			(font
@@
 	(hierarchical_label "spk_on"
 		(shape output)
-		(at 63.5 66.04 180)
-		(effects
-			(font
-				(size 1.27 1.27)
-			)
-			(justify right)
+		(at 63.5 68.58 180)
+		(effects
+			(font
+				(size 1.27 1.27)
+			)
+			(justify right)
+		)
+	)
+	(hierarchical_label "scl"
+		(shape output)
+		(at 134.62 27.94 0)
+		(effects
+			(font
+				(size 1.27 1.27)
+			)
+			(justify left)
 		)
 	)
@@
 	(hierarchical_label "adc_sel1"
 		(shape output)
-		(at 63.5 76.2 180)
+		(at 63.5 63.5 180)
 		(effects
 			(font
@@
 		)
 	)
-	(hierarchical_label "dbgio3"
+	(hierarchical_label "sda"
 		(shape output)
 		(at 134.62 149.86 0)
@@
 		)
 	)
-	(hierarchical_label "edid_clk"
+	(hierarchical_label "scl"
 		(shape output)
 		(at 134.62 147.32 0)
@@
 	(hierarchical_label "uart2_rx"
 		(shape input)
-		(at 63.5 63.5 180)
+		(at 63.5 73.66 180)
 		(effects
 			(font
@@
 	(hierarchical_label "uart_tx"
 		(shape output)
-		(at 63.5 68.58 180)
+		(at 63.5 76.2 180)
 		(effects
 			(font
@@
 		)
 	)
-	(hierarchical_label "dbgio3"
+	(hierarchical_label "sda"
 		(shape output)
 		(at 134.62 78.74 0)
@@
 	(hierarchical_label "uart2_tx"
 		(shape output)
-		(at 63.5 60.96 180)
+		(at 63.5 71.12 180)
 		(effects
 			(font
@@
 	(hierarchical_label "uart_rx"
 		(shape input)
-		(at 63.5 71.12 180)
+		(at 63.5 78.74 180)
 		(effects
 			(font
@@
 		(exclude_from_sim no)
 		(in_bom yes)
-		(on_board yes)
+		(on_board no)
 		(in_pos_files yes)
-		(dnp no)
+		(dnp yes)
 		(fields_autoplaced yes)
 		(property "Reference" "U7"

Commit message: I2C用Groveコネクタを追加
Connections:
- net rgbled: now also U1.47 (PIN86_IOT8A); no longer U1.48 (PIN63_IOR5A)
- net scl: now also U1.48 (PIN63_IOR5A); no longer U1.47 (PIN86_IOT8A)
Changed lines of the file:
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@@
 	(hierarchical_label "scl"
 		(shape output)
-		(at 134.62 27.94 0)
+		(at 134.62 25.4 0)
 		(effects
 			(font
@@
 	(hierarchical_label "rgbled"
 		(shape output)
-		(at 134.62 25.4 0)
+		(at 134.62 27.94 0)
 		(effects
 			(font
